Commit message: adding camera to burger

File: turtlebot3_gazebo/urdf/turtlebot3_burger.urdf (robot description, URDF)
Before this commit: robot turtlebot3_burger, 7 links, 6 joints
Links:
- added link camera_link, mass 0.001; collision box size=.01 .01 .01; visual box size=.02 .02 .02
- added link camera_link_optical
Joints:
- added joint camera_joint: type fixed, parent base_link, child camera_link, origin xyz=0.03 0 0.11 rpy=0 0.79 0, axis 0 1 0
- added joint camera_optical_joint: type fixed, parent camera_link, child camera_link_optical, origin xyz=0 0 0 rpy=-1.57 0 -1.57

Commit message: fix problems with inertia and other parameters so burger is not dancing anymore

File: turtlebot3_gazebo/urdf/turtlebot3_burger.urdf (robot description, URDF)
Before this commit: robot turtlebot3_burger, 9 links, 8 joints
Joints:
- joint camera_joint: origin xyz=0.03 0 0.11 rpy=0 0.79 0 -> xyz=0.03 0 0.11 rpy=0 0.524 0
